File: PCBs/Lab2/mood_ring.sch (EAGLE design)
At the start: 8 parts

Commit message: Changed MSP430 part from through-hole to SMD
Parts:
- U$2: value MSP430G2XX3PDIP -> MSP430G2XX3TSSOP; device ELEC327:MSP430G2XX3PDIP -> ELEC327:MSP430G2XX3TSSOP
Changed lines of the file:
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@@
 <setting verticaltext="up"/>
 </settings>
-<grid distance="0.1" unitdist="inch" unit="inch" style="lines" multiple="1" display="yes" altdistance="0.01" altunitdist="inch" altunit="inch"/>
+<grid distance="0.1" unitdist="inch" unit="inch" style="lines" multiple="1" display="no" altdistance="0.01" altunitdist="inch" altunit="inch"/>
 <layers>
 <layer number="1" name="Top" color="4" fill="1" visible="no" active="no"/>
@@
 </classes>
 <parts>
-<part name="U$2" library="ELEC327" deviceset="MSP430G2XX3" device="PDIP"/>
+<part name="U$2" library="ELEC327" deviceset="MSP430G2XX3" device="TSSOP" value="MSP430G2XX3TSSOP"/>
 <part name="JP1" library="SparkFun" deviceset="M04" device="LOCK"/>
 <part name="R1" library="resistor" deviceset="R-US_" device="R1206"/>
