File: PCBs/Simon-2026-JLC/Simon-2026-JLC.kicad_sch (KiCad schematic)
At the start: 13 parts, among them IC2 MSPM0G3507SPTR, J1 Conn_01x09, J2 Conn_01x05, SW6 SW_SPDT, U1 LIS2HH12

Commit message: Simon PCB 2026
Parts:
- removed SW6: SW_SPDT, Button_Switch_SMD:SW_DPDT_CK_JS202011JCQN, symbol Switch:SW_SPDT
- added C3: 100uF, Capacitor_SMD:C_1206_3216Metric, symbol Device:C
- added SW5: SW_SPDT, ELEC327-Kicad:SW_EG1270, symbol Switch:SW_SPDT
- BT1: footprint Battery:BatteryHolder_Keystone_2468_2xAAA -> Battery:BatteryHolder_Keystone_1060_1x2032; LCSC Part # (none) -> C7498148; MPN (none) -> C7498148
- BZ1: footprint Buzzer_Beeper:Buzzer_CUI_CPT-9019S-SMT -> Buzzer_Beeper:Buzzer_Murata_PKLCS1212E; LCSC Part # (none) -> C113159
- C1: footprint Capacitor_SMD:C_1206_3216Metric_Pad1.33x1.80mm_HandSolder -> Capacitor_SMD:C_0603_1608Metric; LCSC Part # (none) -> C19702
- C2: LCSC Part # (none) -> C1591
- C4: footprint Capacitor_SMD:C_0603_1608Metric_Pad1.08x0.95mm_HandSolder -> Capacitor_SMD:C_0805_2012Metric; LCSC Part # (none) -> C13967
- C6: renamed from C3; footprint Capacitor_SMD:C_0603_1608Metric_Pad1.08x0.95mm_HandSolder -> Capacitor_SMD:C_0402_1005Metric; LCSC Part # (none) -> C15195
- IC2: LCSC Part # (none) -> C22362630
- J1: now not fitted
- J2: LCSC Part # (none) -> C492413
- R5: footprint Resistor_SMD:R_0603_1608Metric_Pad0.98x0.95mm_HandSolder -> Resistor_SMD:R_0603_1608Metric; LCSC Part # (none) -> C105579
- R6: footprint Resistor_SMD:R_0603_1608Metric_Pad0.98x0.95mm_HandSolder -> Resistor_SMD:R_0402_1005Metric; LCSC Part # (none) -> C60491
- U1: LCSC Part # (none) -> C221446
Connections:
- net GND: now also C3.2
- net VDD: now also C3.1, SW5.1 (A)
- net at BT1.1 (+): now also SW5.2 (B)
