File: PCBs/Simon-2026-JLC/simon_io.kicad_sch (KiCad schematic)
At the start: 8 parts, among them SW1 SW_DPST, SW2 SW_DPST, SW3 SW_DPST, SW4 SW_DPST

Commit message: Simon PCB 2026
Parts:
- removed SW1, SW2, SW3, SW4: SW_DPST, Button_Switch_SMD:SW_SPST_PTS645, symbol Switch:SW_DPST
- added SW1, SW2, SW3, SW4: SW_SPST, Button_Switch_SMD:SW_SPST_PTS647_Sx38, symbol Switch:SW_SPST
- LED1, LED2, LED3, LED4: value BL-HBGR32L-3-TRB-8 -> SK9822; footprint BL-HBGR32L-3-TRB-8_AMB -> LED_SMD:LED_RGB_5050-6; LCSC Part # (none) -> C2829089
Connections:
- net BUTTON1_IO: now also SW1.1 (A)
- net BUTTON2_IO: now also SW2.1 (A)
- net BUTTON3_IO: now also SW3.1 (A)
- net BUTTON4_IO: now also SW4.1 (A)
- net GND: now also SW1.2 (B), SW2.2 (B), SW3.2 (B), SW4.2 (B)
